File: lolin-prototype.kicad_pcb (KiCad board)
At the start: 2 copper layers, 83.8 x 78.6 mm, 9 parts, among them J1 BATTERY, J2 LEFT-CONN, J3 RIGHT-CONN, J4 proto-space, J5 I2C, U1 LOLIN32-LITE

Commit message: Trivial updates to make version 1.0
Routing:
- net Net-(BT1-Pad2): track 37.9 -> 39.4 mm
- added copper zone on F.Cu, net GND
- added copper zone on F.Cu, net Net-(BT1-Pad1)
Other:
- board text added: "+"
- board text added: "-"
- board text added: "BATTERY"
- board text added: "FN"
- board text added: "I2C"
- board text added: "IO0"
- board text added: "IO12"
- board text added: "IO13"
- board text added: "IO14"
- board text added: "IO15"
- board text added: "IO16"
- board text added: "IO17"
- board text added: "IO18"
- board text added: "IO19"
- board text added: "IO2"
- board text added: "IO22"
- board text added: "IO23"
- board text added: "IO25"
- board text added: "IO26"
- board text added: "IO27"
- board text added: "IO32"
- board text added: "IO33"
- board text added: "IO34"
- board text added: "IO35"
- board text added: "IO4"
- board text added: "IO5"
- board text added: "Lolin32-Lite Prototype Board"
- board text added: "SCL"
- board text added: "SDA"
- board text added: "VN"
- board text added: "VP"
- board text added: "Version 1.0 by John Spencer, 2017 https://github.com/mage0r/Lolin-Prototype License TAPR OHL v1.0"

Commit message: Updated lolin32-lite and prototyping space footprint
Parts:
- J4: footprint libs:proto-12x12 -> libs:proto-board
- moved J4 0.26 mm to (82.7, 111.3)
Routing:
- net (no net): track 0.00 -> 284.5 mm
- net +3V3: track 127.5 -> 124.3 mm
- net Net-(BT1-Pad2): track 39.4 -> 38.3 mm
