File: lolin-prototype.sch (KiCad schematic (older format))
At the start: 9 parts, among them J1 BATTERY, J2 LEFT-CONN, J3 RIGHT-CONN, J4 proto-space, J5 I2C, U1 LOLIN32-LITE

Commit message: Trivial updates to make version 1.0
Parts:
- R1, R2: renamed from R?; footprint (none) -> Resistors_SMD:R_0603_HandSoldering
Changed lines of the file:
@@
 	6800 2900 6800 2950
 $Comp
-L R R?
+L R R1
 U 1 1 59E0B9C4
 P 6800 2400
-F 0 "R?" V 6880 2400 50  0000 C CNN
+F 0 "R1" V 6880 2400 50  0000 C CNN
 F 1 "1K" V 6800 2400 50  0000 C CNN
-F 2 "" V 6730 2400 50  0001 C CNN
+F 2 "Resistors_SMD:R_0603_HandSoldering" V 6730 2400 50  0001 C CNN
 F 3 "" H 6800 2400 50  0001 C CNN
 	1    6800 2400
@@
 $EndComp
 $Comp
-L R R?
+L R R2
 U 1 1 59E0BA84
 P 7000 2400
-F 0 "R?" V 7080 2400 50  0000 C CNN
+F 0 "R2" V 7080 2400 50  0000 C CNN
 F 1 "1K" V 7000 2400 50  0000 C CNN
-F 2 "" V 6930 2400 50  0001 C CNN
+F 2 "Resistors_SMD:R_0603_HandSoldering" V 6930 2400 50  0001 C CNN
 F 3 "" H 7000 2400 50  0001 C CNN
 	1    7000 2400

Commit message: Updated lolin32-lite and prototyping space footprint
Parts:
- J4: footprint libs:proto-12x12 -> libs:proto-board
Changed lines of the file:
@@
 F 0 "J4" H 6350 1400 50  0000 C CNN
 F 1 "proto-space" V 6450 1250 50  0000 C CNN
-F 2 "libs:proto-12x12" H 6350 1250 50  0001 C CNN
+F 2 "libs:proto-board" H 6350 1250 50  0001 C CNN
 F 3 "" H 6350 1250 50  0001 C CNN
 	1    6350 1250
